File: EagleCAD/TS1.2 04-30-19/Testing suite 1 layout.brd (EAGLE design)
At the start: 71.8 x 58.4 mm, 112 parts

Commit message: Generated gerber file and sent for print. -ATT
Parts:
- moved U$16 7.71 mm to (28.8, 22.7)
- moved U$15 6.67 mm to (28.8, 25.7)
- moved U$3 0.52 mm to (46.7, 20.4)
- moved U$4 0.25 mm to (43.4, 20.4)
Routing:
- net N$7: track 31.5 -> 44.7 mm
- net N$85: track 57.6 -> 66.1 mm
- net N$6: track 38.6 -> 46.2 mm
- net N$11: track 162.9 -> 162.3 mm
Other:
- board text added: "April 30th, 2019"
- board text added: "Baja SAE at Virginia Tech"
- board text added: "By: Matt Herrity"
- board text added: "FL"
- board text added: "FR"
- board text added: "I2C SDA SLC DGND 3.3V"
- board text added: "RL"
- board text added: "RR"
- board text added: "Testing Suite 1.2"
- board text removed: "4/30/2019"
- board text removed: "BAJA VT"
- board text removed: "I2C"
- board text removed: "Matt Herrity"
- board text removed: "Testing Suite 1."
